File: kicad/X1-01M-carrier/X1-01M-carrier.kicad_pcb (KiCad board)
At the start: 2 copper layers, 48.9 x 78.7 mm, 13 parts, among them J1 AudioJack4, J2 Conn_01x02, J3 Conn_Coaxial, SW1 SW_SPDT, SW2 Push Button, U1 USB-C-Power_Only, U2 XL01M

Commit message: added docs, added gerber, finished layout
Parts:
- moved U1 1.32 mm to (147.0, 128.7)
- moved J1 1.08 mm to (125.1, 125.4)
- moved SW1 0.52 mm to (135.7, 131.7)
- moved C3 0.52 mm to (141.2, 119.7)
- moved J2 0.52 mm to (130.0, 99.1)
- moved D1 0.52 mm to (131.0, 58.5)
- moved C1 0.52 mm to (121.5, 118.5)
- moved C2 0.52 mm to (128.5, 118.5)
- moved U2 0.52 mm to (133.0, 104.5)
- moved SW2 0.52 mm to (120.8, 58.8)
- moved C4 0.52 mm to (145.1, 119.7)
- moved L1 0.52 mm to (141.2, 112.7)
- moved J3 0.42 mm to (151.5, 60.7)
Routing:
- net Net-(U2-Right_Channel): track 0.00 -> 25.3 mm
- net Net-(D1-A): track 16.4 -> 39.3 mm
- net +5V: track 11.2 -> 23.1 mm
- net Net-(U2-Left_Channel): track 14.9 -> 26.5 mm
- net Net-(J2-Pin_2): track 38.1 -> 48.3 mm
- net Net-(J2-Pin_1): track 37.3 -> 45.6 mm
- net Net-(C1-Pad2): track 7.33 -> 6.66 mm
- net Net-(SW1-B): track 17.9 -> 18.6 mm
- net GND: vias 0 -> 380
Other:
- board size 48.9 x 78.7 mm -> 47.4 x 78.7 mm
